Commit message: Added workcell geometry; added vacuum gripper geometry and plugin; added bin geometry and plugin; added kinect plugin

File: gilbreth_support/urdf/gilbreth.xacro (robot description, xacro)
@@ -1,4 +1,4 @@
 <?xml version="1.0" ?>
-<robot name="gilbreth" xmlns:xacro="http://ros.org/wiki/xacro">
+<robot name="gilbreth" xmlns:xacro="http://www.ros.org/wiki/xacro">
   <!-- include the robot xacro -->
   <xacro:include filename="$(find ur_description)/urdf/ur10.urdf.xacro" />
@@ -11,28 +11,56 @@
   <xacro:include filename="$(find gilbreth_support)/urdf/linear_actuator/linear_actuator.xacro" />
   <xacro:linear_actuator prefix="linear_actuator_"/>
+  <!-- bins -->
+  <xacro:include filename="$(find gilbreth_support)/urdf/bin/bin.xacro"/>
+  <xacro:bin prefix="bin_1_"/>
+  <xacro:bin prefix="bin_2_"/>
+  <xacro:bin prefix="bin_3_"/>
+  <!-- depth camera -->
+  <xacro:include filename="$(find gilbreth_support)/urdf/depth_camera/depth_camera.xacro"/>
+  <xacro:depth_camera prefix="rgbd_1_"/>
   <!-- Links -->
-  <link name="world" />
-  <link name="break_beam_frame" />
-  <link name="camera_link" />
-  <link name="bin1_frame" />
-  <link name="bin2_frame" />
-  <link name="bin3_frame" />
-  <link name="bin4_frame" />
-  <link name="bin5_frame" />
-  <link name="bin6_frame" />
-  <link name="bin7_frame" />
-  <link name="bin8_frame" />
-  <link name="agv1_load_point_frame" />
-  <link name="agv2_load_point_frame" />
-  <link name="belt_frame" />
+  <link name="world"/>
+  <link name="test_link">
+    <visual>
+      <geometry>
+        <mesh filename="package://gilbreth_support/meshes/workcell/visual/workcell.dae"/>
+      </geometry>
+    </visual>
+    <collision>
+      <geometry>
+        <mesh filename="package://gilbreth_support/meshes/workcell/collision/workcell.ply"/>
+      </geometry>
+    </collision>
+    <inertial>
+      <inertia ixx="1.0" ixy="0" ixz="0"
+               iyy="1.0" iyz="0"
+               izz="1.0" />
+      <mass value="100" />
+    </inertial>
+  </link>
+  <link name="conveyor_dummy_link"/>
+  <link name="break_beam" />
   <!-- Joints -->
-  <joint name="world_to_linear_actuator" type="fixed">
+  <joint name="test_joint" type="fixed">
     <parent link="world" />
+    <child link="test_link" />
+    <dynamics friction="1000" damping="1.0"/>
+  </joint>
+  <joint name="conveyor_dummy_to_world" type="fixed">
+    <parent link="test_link" />
+    <child link="conveyor_dummy_link" />
+    <origin xyz="0 -1.2 0.9" rpy="0 0 -${radians(90)}" />
+    <dynamics friction="1000" damping="1.0"/>
+  </joint>
+  <joint name="conveyor_dummy_to_linear_actuator" type="fixed">
+    <parent link="conveyor_dummy_link" />
     <child link="linear_actuator_base_link" />
-    <origin xyz="0.3 0.0 0.9" rpy="0.0 0.0 0.0" />
+    <origin xyz="-0.8 0 0" rpy="0 0 0" />
+    <dynamics friction="1000" damping="1.0"/>
   </joint>
   <joint name="robot_to_actuator_carriage" type="fixed">
     <parent link="linear_actuator_carriage" />
     <child link="robot_base_link" />
+    <dynamics friction="5000" damping="1.0"/>
   </joint>
   <joint name="vacuum_gripper_to_robot" type="fixed">
@@ -42,77 +70,31 @@
   <!-- a break_beam type sensor in the frame break_beam_frame -->
   <joint name="break_beam_joint" type="fixed">
-    <parent link="world" />
-    <child link="break_beam_frame" />
-    <origin xyz="1.6 3.5 0.91" rpy="0 0 ${pi}" />
+    <parent link="conveyor_dummy_link" />
+    <child link="break_beam" />
+    <origin xyz="0.0 3.5 0.75" rpy="0 0 ${pi}" />
   </joint>
   <!-- a kinect camera in the frame kinect_camera_frame -->
   <joint name="camera_link" type="fixed">
-    <parent link="world"/>
-    <child link="camera_link" />
-    <origin xyz="1.21 3.0 1.66" rpy="${pi} 0 -${pi/2}" />
+    <parent link="conveyor_dummy_link"/>
+    <child link="rgbd_1_base_link" />
+    <origin xyz="0.0 3.0 0.75" rpy="${pi/2} ${pi/2} 0" />
   </joint>
   <!-- a bin in the frame bin1_frame -->
-  <joint name="bin1_joint" type="fixed">
-    <parent link="world" />
-    <child link="bin1_frame" />
-    <origin xyz="-1.0 -1.33 0.72" rpy="0 0 ${pi/2}" />
+  <joint name="bin_1_joint" type="fixed">
+    <parent link="linear_actuator_base_link" />
+    <child link="bin_1_base_link" />
+    <origin xyz="-0.8 -1.0 -0.9" rpy="0 0 0" />
   </joint>
   <!-- a bin in the frame bin2_frame -->
-  <joint name="bin2_joint" type="fixed">
-    <parent link="world" />
-    <child link="bin2_frame" />
-    <origin xyz="-1.0 -0.535 0.72" rpy="0 0 ${pi/2}" />
+  <joint name="bin_2_joint" type="fixed">
+    <parent link="linear_actuator_base_link" />
+    <child link="bin_2_base_link" />
+    <origin xyz="-0.8 0.0 -0.9" rpy="0 0 0" />
   </joint>
   <!-- a bin in the frame bin3_frame -->
-  <joint name="bin3_joint" type="fixed">
-    <parent link="world" />
-    <child link="bin3_frame" />
-    <origin xyz="-1.0 0.23 0.72" rpy="0 0 ${pi/2}" />
-  </joint>
-  <!-- a bin in the frame bin4_frame -->
-  <joint name="bin4_joint" type="fixed">
-    <parent link="world" />
-    <child link="bin4_frame" />
-    <origin xyz="-1.0 0.995 0.72" rpy="0 0 ${pi/2}" />
-  </joint>
-  <!-- a bin in the frame bin5_frame -->
-  <joint name="bin5_joint" type="fixed">
-    <parent link="world" />
-    <child link="bin5_frame" />
-    <origin xyz="-0.3 -1.33 0.72" rpy="0 0 ${pi/2}" />
-  </joint>
-  <!-- a bin in the frame bin6_frame -->
-  <joint name="bin6_joint" type="fixed">
-    <parent link="world" />
-    <child link="bin6_frame" />
-    <origin xyz="-0.3 -0.535 0.72" rpy="0 0 ${pi/2}" />
-  </joint>
-  <!-- a bin in the frame bin7_frame -->
-  <joint name="bin7_joint" type="fixed">
-    <parent link="world" />
-    <child link="bin7_frame" />
-    <origin xyz="-0.3 0.23 0.72" rpy="0 0 ${pi/2}" />
-  </joint>
-  <!-- a bin in the frame bin8_frame -->
-  <joint name="bin8_joint" type="fixed">
-    <parent link="world" />
-    <child link="bin8_frame" />
-    <origin xyz="-0.3 0.995 0.72" rpy="0 0 ${pi/2}" />
-  </joint>
-  <!-- agv load point frames -->
-  <joint name="agv1_load_point_joint" type="fixed">
-    <parent link="world" />
-    <child link="agv1_load_point_frame" />
-    <origin xyz="0.3 3.3 0.75" rpy="0 0 ${pi}" />
-  </joint>
-  <joint name="agv2_load_point_joint" type="fixed">
-    <parent link="world" />
-    <child link="agv2_load_point_frame" />
-    <origin xyz="0.3 -3.3 0.75" rpy="0 0 0" />
-  </joint>
-  <joint name="belt_joint" type="fixed">
-    <parent link="world" />
-    <child link="belt_frame" />
-    <origin xyz="1.24 0.15 0.91" rpy="0 0 0" />
+  <joint name="bin_3_joint" type="fixed">
+    <parent link="linear_actuator_base_link" />
+    <child link="bin_3_base_link" />
+    <origin xyz="-0.8 1.0 -0.9" rpy="0 0 0" />
   </joint>
   <gazebo>

File: gilbreth_support/urdf/vacuum_gripper/vacuum_gripper.gazebo.xacro (robot description, xacro)
@@ -3,24 +3,24 @@
   <xacro:macro name="vacuum_gripper_gazebo" params="prefix **drops_info">
     <gazebo reference="${prefix}base_link">
-        <material>Gazebo/Red</material>
-      </gazebo>
-      <gazebo reference="${prefix}tool0">
-        <material>Gazebo/Red</material>
-      </gazebo>
-      <gazebo>
-        <plugin name="ros_vacuum_gripper" filename="libROSVacuumGripperPlugin.so">
-          <grasp_check>
-            <detach_steps>40</detach_steps>
-            <attach_steps>1</attach_steps>
-            <min_contact_count>1</min_contact_count>
-          </grasp_check>
-          <xacro:insert_block name="drops_info" />
-          <suction_cup_link>vacuum_gripper_link</suction_cup_link>
-          <!-- ROS -->
-          <robot_namespace>/gilbreth</robot_namespace>
-          <control_topic>gripper/control</control_topic>
-          <state_topic>gripper/state</state_topic>
-        </plugin>
-      </gazebo>
+      <material>Gazebo/Red</material>
+    </gazebo>
+    <gazebo reference="${prefix}tool0">
+      <material>Gazebo/Red</material>
+    </gazebo>
+    <gazebo>
+      <plugin name="ros_vacuum_gripper" filename="libROSVacuumGripperPlugin.so">
+        <grasp_check>
+          <detach_steps>40</detach_steps>
+          <attach_steps>1</attach_steps>
+          <min_contact_count>1</min_contact_count>
+        </grasp_check>
+        <xacro:insert_block name="drops_info" />
+        <suction_cup_link>${prefix}tool0</suction_cup_link>
+        <!-- ROS -->
+        <robot_namespace>/gilbreth</robot_namespace>
+        <control_topic>gripper/control</control_topic>
+        <state_topic>gripper/state</state_topic>
+      </plugin>
+    </gazebo>
   </xacro:macro>
 </robot>

File: gilbreth_support/urdf/vacuum_gripper/vacuum_gripper.urdf.xacro (robot description, xacro)
@@ -1,14 +1,11 @@
 <?xml version="1.0"?>
 <robot xmlns:xacro="http://www.ros.org/wiki/xacro">
-  <xacro:property name="radius" value="0.05"/>
-  <xacro:property name="length" value="0.1"/>
-  <xacro:property name="test" value="${radius*length}"/>
   <xacro:macro name="vacuum_gripper_urdf" params="prefix">
     <!-- link list -->
     <link name="${prefix}base_link">
       <visual>
-        <origin xyz="0 0 ${length / 2}" rpy="0 0 0" />
+        <origin xyz="0 0 0" rpy="0 0 0" />
         <geometry>
-          <cylinder radius="${radius}" length="${length}" />
+          <mesh filename="package://gilbreth_support/meshes/vacuum_gripper/visual/vacuum_gripper.dae"/>
         </geometry>
         <material name="red">
@@ -17,7 +14,7 @@
       </visual>
       <collision>
-        <origin xyz="0 0 ${length / 2}" rpy="0 0 0"/>
+        <origin xyz="0 0 0" rpy="0 0 0"/>
         <geometry>
-          <cylinder radius="${radius}" length="${length}"/>
+          <mesh filename="package://gilbreth_support/meshes/vacuum_gripper/collision/vacuum_gripper.ply"/>
         </geometry>
         <material name="red"/>
@@ -25,8 +22,8 @@
       <inertial>
         <origin xyz="0 0 0" rpy="0 0 0" />
-        <inertia ixx="0.0000063" ixy="0" ixz="0"
-                 iyy="0.0000063" iyz="0"
-                 izz="0.000025" />
-        <mass value="0.01" />
+        <inertia ixx="1.0" ixy="0" ixz="0"
+                 iyy="1.0" iyz="0"
+                 izz="1.0" />
+        <mass value="1.0" />
       </inertial>
     </link>
@@ -34,5 +31,5 @@
     <!-- joint list -->
     <joint name="vacuum_gripper_joint" type="fixed">
-      <origin xyz="0 0 ${length}" rpy="0 0 0" />
+      <origin xyz="0 0 0.080" rpy="0 0 0" />
       <parent link="${prefix}base_link" />
       <child link="${prefix}tool0" />

Commit message: Fixes to MoveIt config; prefix naming change in spawn launch to allow Gazebo controller to work for move group

File: gilbreth_support/urdf/gilbreth.xacro (robot description, xacro)
@@ -2,12 +2,6 @@
 <robot name="gilbreth" xmlns:xacro="http://www.ros.org/wiki/xacro">
   <!-- linear arm actuator -->
-  <xacro:include filename="$(find gilbreth_support)/urdf/linear_actuator/linear_actuator.urdf.xacro" />
+  <xacro:include filename="$(find gilbreth_support)/urdf/linear_actuator/linear_actuator.urdf.xacro"/>
   <xacro:linear_actuator_urdf prefix="linear_actuator_"/>
-  <!-- include the robot xacro -->
-<!--  <xacro:include filename="$(find ur_description)/urdf/ur10.urdf.xacro" />
-  <xacro:ur10_robot prefix="robot_" joint_limited="false"/>-->
-  <!-- vacuum gripper -->
-<!--  <xacro:include filename="$(find gilbreth_support)/urdf/vacuum_gripper/vacuum_gripper.urdf.xacro"/>
-  <xacro:vacuum_gripper_urdf prefix="vacuum_gripper_"/>-->
   <!-- bins -->
 <!--  <xacro:include filename="$(find gilbreth_support)/urdf/bin/bin.xacro"/>
@@ -27,16 +21,4 @@
     <parent link="world" />
     <child link="world_interface" />
-  </joint>
-<!--  <joint name="linear_actuator_to_workcell" type="fixed">
-    <parent link="world" />
-    <child link="linear_actuator_world_interface" />
-  </joint>-->
-  <joint name="robot_to_actuator_carriage" type="fixed">
-    <parent link="linear_actuator_carriage" />
-    <child link="robot_base_link" />
-  </joint>
-  <joint name="vacuum_gripper_to_robot" type="fixed">
-    <parent link="robot_tool0" />
-    <child link="vacuum_gripper_base_link" />
   </joint>
   <!-- a break_beam type sensor in the frame break_beam_frame -->
@@ -68,3 +50,8 @@
     <origin xyz="-0.8 1.0 -0.9" rpy="0 0 0" />
   </joint>-->
+<!--  <gazebo>
+    <plugin name="gazebo_ros_control" filename="libgazebo_ros_control.so">
+      <robotNamespace>/</robotNamespace>
+    </plugin>
+  </gazebo>-->
 </robot>

File: gilbreth_support/urdf/linear_actuator/linear_actuator.gazebo.xacro (robot description, xacro)
@@ -8,7 +8,4 @@
       <material>Gazebo/Grey</material>
     </gazebo>
-<!--    <gazebo reference="${prefix}carriage_joint">
-      <implicitSpringDamper>1</implicitSpringDamper>
-    </gazebo>-->
     <transmission name="${prefix}transmission">
       <type>transmission_interface/SimpleTransmission</type>
@@ -21,7 +18,6 @@
     </transmission>
     <gazebo>
-<!--      <static>true</static>-->
       <plugin name="gazebo_ros_control" filename="libgazebo_ros_control.so">
-        <robotNamespace>gilbreth</robotNamespace>
+        <robotNamespace>/</robotNamespace>
         <robotParam>${prefix}description</robotParam>
       </plugin>

File: gilbreth_support/urdf/linear_actuator/linear_actuator.urdf.xacro (robot description, xacro)
@@ -1,4 +1,8 @@
 <?xml version="1.0"?>
 <robot name="linear_actuator_urdf" xmlns:xacro="http://www.ros.org/wiki/xacro">
+  <xacro:include filename="$(find ur_description)/urdf/ur10.urdf.xacro"/>
+  <xacro:ur10_robot prefix="robot_" joint_limited="true"/>
+  <xacro:include filename="$(find gilbreth_support)/urdf/vacuum_gripper/vacuum_gripper.urdf.xacro"/>
+  <xacro:vacuum_gripper_urdf prefix="vacuum_gripper_"/>
   <xacro:macro name="linear_actuator_urdf" params="prefix">
     <xacro:property name="width" value="0.2" />
@@ -6,8 +10,4 @@
     <xacro:property name="height" value="0.1" />
     <xacro:property name="carriage_length" value="0.2"/>
-    <xacro:include filename="$(find ur_description)/urdf/ur10.urdf.xacro"/>
-    <xacro:ur10_robot prefix="robot_" joint_limited="false"/>
-    <xacro:include filename="$(find gilbreth_support)/urdf/vacuum_gripper/vacuum_gripper.urdf.xacro"/>
-    <xacro:vacuum_gripper_urdf prefix="vacuum_gripper_"/>
     <!-- link list -->
     <link name="world"/>

File: gilbreth_support/urdf/linear_actuator/linear_actuator.xacro (robot description, xacro)
@@ -7,4 +7,4 @@
   <!-- Gazebo -->
   <xacro:include filename="$(find gilbreth_support)/urdf/linear_actuator/linear_actuator.gazebo.xacro"/>
-  <xacro:linear_actuator_gazebo prefix="$(arg prefix)" joint_interface="hardware_interface/PositionJointInterface"/>
+  <xacro:linear_actuator_gazebo prefix="$(arg prefix)" joint_interface="PositionJointInterface"/>
 </robot>

Commit message: Added gripper link input argument to vacuum gripper gazebo xacro; made a new xacro for the combine robot system (robot, rail, gripper)

File: gilbreth_support/urdf/gilbreth.xacro (robot description, xacro)
@@ -1,7 +1,6 @@
 <?xml version="1.0" ?>
 <robot name="gilbreth" xmlns:xacro="http://www.ros.org/wiki/xacro">
-  <!-- linear arm actuator -->
-  <xacro:include filename="$(find gilbreth_support)/urdf/linear_actuator/linear_actuator.urdf.xacro"/>
-  <xacro:linear_actuator_urdf prefix="linear_actuator_"/>
+  <!-- robot system -->
+  <xacro:include filename="$(find gilbreth_support)/urdf/robot_system/robot_system.xacro"/>
   <!-- bins -->
 <!--  <xacro:include filename="$(find gilbreth_support)/urdf/bin/bin.xacro"/>
@@ -50,8 +49,3 @@
     <origin xyz="-0.8 1.0 -0.9" rpy="0 0 0" />
   </joint>-->
-<!--  <gazebo>
-    <plugin name="gazebo_ros_control" filename="libgazebo_ros_control.so">
-      <robotNamespace>/</robotNamespace>
-    </plugin>
-  </gazebo>-->
 </robot>

File: gilbreth_support/urdf/linear_actuator/linear_actuator.gazebo.xacro (robot description, xacro)
@@ -17,10 +17,4 @@
       </actuator>
     </transmission>
-    <gazebo>
-      <plugin name="gazebo_ros_control" filename="libgazebo_ros_control.so">
-        <robotNamespace>/</robotNamespace>
-        <robotParam>${prefix}description</robotParam>
-      </plugin>
-    </gazebo>
   </xacro:macro>
 </robot>

File: gilbreth_support/urdf/linear_actuator/linear_actuator.urdf.xacro (robot description, xacro)
@@ -1,8 +1,4 @@
 <?xml version="1.0"?>
 <robot name="linear_actuator_urdf" xmlns:xacro="http://www.ros.org/wiki/xacro">
-  <xacro:include filename="$(find ur_description)/urdf/ur10.urdf.xacro"/>
-  <xacro:ur10_robot prefix="robot_" joint_limited="true"/>
-  <xacro:include filename="$(find gilbreth_support)/urdf/vacuum_gripper/vacuum_gripper.urdf.xacro"/>
-  <xacro:vacuum_gripper_urdf prefix="vacuum_gripper_"/>
   <xacro:macro name="linear_actuator_urdf" params="prefix">
     <xacro:property name="width" value="0.2" />
@@ -63,12 +59,4 @@
       <dynamics damping="0.7" friction="500.0" />
     </joint>
-    <joint name="${prefix}joint_2" type="fixed">
-      <parent link="${prefix}carriage" />
-      <child link="robot_base_link" />
-    </joint>
-    <joint name="${prefix}joint_3" type="fixed">
-      <parent link="robot_tool0" />
-      <child link="vacuum_gripper_base_link" />
-    </joint>
   </xacro:macro>
 </robot>

File: gilbreth_support/urdf/vacuum_gripper/vacuum_gripper.gazebo.xacro (robot description, xacro)
@@ -1,5 +1,5 @@
 <?xml version="1.0"?>
 <robot xmlns:xacro="http://www.ros.org/wiki/xacro">
-  <xacro:macro name="vacuum_gripper_gazebo" params="prefix **drops_info">
+  <xacro:macro name="vacuum_gripper_gazebo" params="prefix **drops_info gripper_link">
     <gazebo reference="${prefix}base_link">
       <material>Gazebo/Red</material>
@@ -16,5 +16,5 @@
         </grasp_check>
         <xacro:insert_block name="drops_info" />
-        <suction_cup_link>${prefix}::${prefix}base_link</suction_cup_link>
+        <suction_cup_link>${gripper_link}</suction_cup_link>
         <!-- ROS -->
         <robot_namespace>/gilbreth</robot_namespace>

File: gilbreth_support/urdf/vacuum_gripper/vacuum_gripper.xacro (robot description, xacro)
@@ -7,5 +7,5 @@
   <!-- Gazebo -->
   <xacro:include filename="$(find gilbreth_support)/urdf/vacuum_gripper/vacuum_gripper.gazebo.xacro"/>
-  <xacro:vacuum_gripper_gazebo prefix="$(arg prefix)">
+  <xacro:vacuum_gripper_gazebo prefix="$(arg prefix)" gripper_link="${prefix}::${prefix}tool0">
     <drops_info/>
   </xacro:vacuum_gripper_gazebo>
