Commit message: Minor changes per PR review; moved ReadMe to top level

File: gilbreth_support/urdf/vacuum_gripper/vacuum_gripper.urdf.xacro (robot description, xacro)
@@ -28,13 +28,5 @@
       </inertial>
     </link>
-    <link name="${prefix}tool0">
-<!--      <inertial>
-        <origin xyz="0 0 0" rpy="0 0 0" />
-        <inertia ixx="0.1" ixy="0" ixz="0"
-                 iyy="0.1" iyz="0"
-                 izz="0.1" />
-        <mass value="1" />
-      </inertial>-->
-    </link>
+    <link name="${prefix}tool0"/>
     <!-- joint list -->
     <joint name="vacuum_gripper_joint" type="fixed">

File: gilbreth_support/urdf/workcell/workcell.xacro (robot description, xacro)
@@ -2,13 +2,5 @@
 <robot name="workcell" xmlns:xacro="http://www.ros.org/wiki/xacro">
   <!-- Links -->
-  <link name="world_interface">
-<!--    <inertial>
-      <origin xyz="0 0 0" rpy="0 0 0" />
-      <inertia ixx="0.1" ixy="0" ixz="0"
-               iyy="0.1" iyz="0"
-               izz="0.1" />
-      <mass value="1" />
-    </inertial>-->
-  </link>
+  <link name="world_interface"/>
   <link name="workcell">
     <visual>

Commit message: Changed vacuum gripper end link from tool0 to suction cup per comment by gavanderhoorn

File: gilbreth_support/urdf/vacuum_gripper/vacuum_gripper.urdf.xacro (robot description, xacro)
@@ -28,10 +28,10 @@
       </inertial>
     </link>
-    <link name="${prefix}tool0"/>
+    <link name="${prefix}suction_cup"/>
     <!-- joint list -->
     <joint name="vacuum_gripper_joint" type="fixed">
       <origin xyz="0 0 0.080" rpy="0 0 0" />
       <parent link="${prefix}base_link" />
-      <child link="${prefix}tool0" />
+      <child link="${prefix}suction_cup" />
     </joint>
   </xacro:macro>
