Commit message: Changes to conveyor spawner models

File: gilbreth_support/urdf/conveyor_objects/disk.xacro (robot description, xacro)
@@ -1,41 +1,5 @@
 <?xml version="1.0"?>
 <robot name="disk" xmlns:xacro="http://www.ros.org/wiki/xacro">
-  <!-- link list -->
-  <link name="base_link">
-    <visual>
-      <origin xyz="0 0 0" rpy="0 0 0" />
-      <geometry>
-        <mesh filename="package://gilbreth_support/meshes/conveyor_objects/visual/disk.stl" />
-      </geometry>
-      <material name="dark_grey">
-        <color rgba="0.1 0.1 0.1 1.0"/>
-      </material>
-    </visual>
-    <collision>
-      <origin xyz="0 0 0" rpy="0 0 0" />
-      <geometry>
-        <mesh filename="package://gilbreth_support/meshes/conveyor_objects/collision/disk.stl" />
-      </geometry>
-      <material name="dark_grey"/>
-      <surface>
-        <friction>
-          <ode>
-            <mu>1.0</mu>
-            <mu2>1.0</mu2>
-          </ode>
-          <torsional>
-            <coefficient>1000.0</coefficient>
-            <patch_radius>0.1</patch_radius>
-          </torsional>
-        </friction>
-      </surface>
-    </collision>
-    <inertial>
-      <origin xyz="0 0 0" rpy="0 0 0" />
-      <inertia ixx="0.1" ixy="0" ixz="0"
-               iyy="0.1" iyz="0"
-               izz="0.1" />
-      <mass value="1" />
-    </inertial>
-  </link>
+  <xacro:include filename="$(find gilbreth_support)/urdf/conveyor_objects/disk_macro.xacro"/>
+  <xacro:disk prefix="disk_"/>
 </robot>

File: gilbreth_support/urdf/conveyor_objects/gasket.xacro (robot description, xacro)
@@ -1,29 +1,5 @@
 <?xml version="1.0"?>
 <robot name="gasket" xmlns:xacro="http://www.ros.org/wiki/xacro">
-  <!-- link list -->
-  <link name="base_link">
-    <visual>
-      <origin xyz="0 0 0" rpy="0 0 0" />
-      <geometry>
-        <mesh filename="package://gilbreth_support/meshes/conveyor_objects/visual/gasket.stl" />
-      </geometry>
-      <material name="dark_grey">
-        <color rgba="0.1 0.1 0.1 1.0"/>
-      </material>
-    </visual>
-    <collision>
-      <origin xyz="0 0 0" rpy="0 0 0" />
-      <geometry>
-        <mesh filename="package://gilbreth_support/meshes/conveyor_objects/collision/gasket.stl" />
-      </geometry>
-      <material name="dark_grey"/>
-    </collision>
-    <inertial>
-      <origin xyz="0 0 0" rpy="0 0 0" />
-      <inertia ixx="0.1" ixy="0" ixz="0"
-               iyy="0.1" iyz="0"
-               izz="0.1" />
-      <mass value="1" />
-    </inertial>
-  </link>
+  <xacro:include filename="$(find gilbreth_support)/urdf/conveyor_objects/gasket_macro.xacro"/>
+  <xacro:gasket prefix="gasket_"/>
 </robot>

File: gilbreth_support/urdf/conveyor_objects/gear.xacro (robot description, xacro)
@@ -1,29 +1,5 @@
 <?xml version="1.0"?>
 <robot name="gear" xmlns:xacro="http://www.ros.org/wiki/xacro">
-  <!-- link list -->
-  <link name="base_link">
-    <visual>
-      <origin xyz="0 0 0" rpy="0 0 0" />
-      <geometry>
-        <mesh filename="package://gilbreth_support/meshes/conveyor_objects/visual/gear.stl" />
-      </geometry>
-      <material name="dark_grey">
-        <color rgba="0.1 0.1 0.1 1.0"/>
-      </material>
-    </visual>
-    <collision>
-      <origin xyz="0 0 0" rpy="0 0 0" />
-      <geometry>
-        <mesh filename="package://gilbreth_support/meshes/conveyor_objects/collision/gear.stl" />
-      </geometry>
-      <material name="dark_grey"/>
-    </collision>
-    <inertial>
-      <origin xyz="0 0 0" rpy="0 0 0" />
-      <inertia ixx="0.1" ixy="0" ixz="0"
-               iyy="0.1" iyz="0"
-               izz="0.1" />
-      <mass value="1" />
-    </inertial>
-  </link>
+  <xacro:include filename="$(find gilbreth_support)/urdf/conveyor_objects/gear_macro.xacro"/>
+  <xacro:gear prefix="gear_"/>
 </robot>

File: gilbreth_support/urdf/conveyor_objects/piston_rod.xacro (robot description, xacro)
@@ -1,29 +1,5 @@
 <?xml version="1.0"?>
 <robot name="piston_rod" xmlns:xacro="http://www.ros.org/wiki/xacro">
-  <!-- link list -->
-  <link name="base_link">
-    <visual>
-      <origin xyz="0 0 0" rpy="0 0 0" />
-      <geometry>
-        <mesh filename="package://gilbreth_support/meshes/conveyor_objects/visual/piston_rod.stl" />
-      </geometry>
-      <material name="dark_grey">
-        <color rgba="0.1 0.1 0.1 1.0"/>
-      </material>
-    </visual>
-    <collision>
-      <origin xyz="0 0 0" rpy="0 0 0" />
-      <geometry>
-        <mesh filename="package://gilbreth_support/meshes/conveyor_objects/collision/piston_rod.stl" />
-      </geometry>
-      <material name="dark_grey"/>
-    </collision>
-    <inertial>
-      <origin xyz="0 0 0" rpy="0 0 0" />
-      <inertia ixx="0.1" ixy="0" ixz="0"
-               iyy="0.1" iyz="0"
-               izz="0.1" />
-      <mass value="1" />
-    </inertial>
-  </link>
+  <xacro:include filename="$(find gilbreth_support)/urdf/conveyor_objects/piston_rod_macro.xacro"/>
+  <xacro:piston_rod prefix="piston_rod_"/>
 </robot>

File: gilbreth_support/urdf/conveyor_objects/pulley.xacro (robot description, xacro)
@@ -1,29 +1,5 @@
 <?xml version="1.0"?>
 <robot name="pulley" xmlns:xacro="http://www.ros.org/wiki/xacro">
-  <!-- link list -->
-  <link name="base_link">
-    <visual>
-      <origin xyz="0 0 0" rpy="0 0 0" />
-      <geometry>
-        <mesh filename="package://gilbreth_support/meshes/conveyor_objects/visual/pulley.stl" />
-      </geometry>
-      <material name="dark_grey">
-        <color rgba="0.1 0.1 0.1 1.0"/>
-      </material>
-    </visual>
-    <collision>
-      <origin xyz="0 0 0" rpy="0 0 0" />
-      <geometry>
-        <mesh filename="package://gilbreth_support/meshes/conveyor_objects/collision/pulley.stl" />
-      </geometry>
-      <material name="dark_grey"/>
-    </collision>
-    <inertial>
-      <origin xyz="0 0 0" rpy="0 0 0" />
-      <inertia ixx="0.1" ixy="0" ixz="0"
-               iyy="0.1" iyz="0"
-               izz="0.1" />
-      <mass value="1" />
-    </inertial>
-  </link>
+  <xacro:include filename="$(find gilbreth_support)/urdf/conveyor_objects/pulley_macro.xacro"/>
+  <xacro:pulley prefix="pulley_"/>
 </robot>
