Commit message: Modified based on new models

File: gilbreth_support/urdf/break_beam/break_beam.gazebo.xacro (robot description, xacro)
@@ -9,7 +9,6 @@
       <sensor name="${prefix}sensor" type="ray">
         <pose>0 0 0 0 0 0</pose>
-        <visualize>true</visualize>
-        <update_rate>10.0</update_rate>
-        <ray>
+<!--        <update_rate>10.0</update_rate> -->
+<!--        <ray>
           <scan>
             <horizontal>
@@ -31,12 +30,37 @@
           </noise>
         </ray>
+-->
         <always_on>1</always_on>
-        <plugin name="${prefix}controller" filename="libgazebo_ros_laser.so" >
-          <topicName>laser/scan</topicName>
-          <frameName>${prefix}optical_link</frameName>
+        <visualize>true</visualize>
+        <plugin name="${prefix}controller" filename="libROSProximityRayPlugin.so" >
+          <robotNamespace>gilbreth</robotNamespace>
+          <time_delay>0.05</time_delay><!-- this modifies the update rate of the ray sensor -->
         </plugin>
+        <ray>
+          <range>
+            <min>0.0</min>
+            <max>1.0</max> <!-- this represents the distance at which the reflector's placed. max 12m -->
+            <resolution>0.001</resolution>
+          </range>
+          <scan>
+            <horizontal>
+              <samples>1</samples>
+              <resolution>1</resolution>
+              <min_angle>0</min_angle>
+              <max_angle>0</max_angle>
+            </horizontal>
+          </scan>
+          <noise>
+            <type>gaussian</type>
+            <mean>0.0</mean>
+            <stddev>0.001</stddev>
+          </noise>
+        </ray>
+        <visualize>true</visualize>
+        <always_on>1</always_on>
       </sensor>
     </gazebo>
     <gazebo>
+      <gravity>false</gravity>
       <static>true</static>
     </gazebo>

File: gilbreth_support/urdf/break_beam/break_beam.urdf.xacro (robot description, xacro)
@@ -34,10 +34,10 @@
       <parent link="${prefix}world_interface" />
       <child link="${prefix}base_link" />
-      <origin xyz="1.2 3.5 1.65" rpy="0 ${radians(90)} -${radians(90)}" />
+      <origin xyz="1.6 2.8 0.925" rpy="0 0 3.14159265359" />
     </joint>
     <joint name="${prefix}joint_1" type="fixed">
       <parent link="${prefix}base_link" />
       <child link="${prefix}optical_link" />
-      <origin xyz="0 0 0.025" rpy="0 0 0" />
+      <origin xyz="0.025 0 0.00" rpy="0 0 0" />
     </joint>
   </xacro:macro>

Commit message: changed the plugin
edited the pose

nothing changed

nothing changed

nothing changed

new header file

nothing changed

new plugins and msgs

new laser plugins

new laser headers

added new plugins and msgs

deleted

nothing changed from origin

Removed unnecessary comments

File: gilbreth_support/urdf/break_beam/break_beam.gazebo.xacro (robot description, xacro)
@@ -16,6 +16,6 @@
               <samples>50</samples>
               <resolution>1</resolution>
-              <min_angle>-${radians(20)}</min_angle>
-              <max_angle>${radians(20)}</max_angle>
+              <min_angle>0</min_angle>
+              <max_angle>0</max_angle>
             </horizontal>
           </scan>
@@ -32,5 +32,5 @@
         </ray>
         <always_on>1</always_on>
-        <plugin name="${prefix}controller" filename="libgazebo_ros_laser.so" >
+        <plugin name="${prefix}controller" filename="libROSProximityRayPlugin.so" >
           <topicName>laser/scan</topicName>
           <frameName>${prefix}optical_link</frameName>

File: gilbreth_support/urdf/break_beam/break_beam.urdf.xacro (robot description, xacro)
@@ -34,5 +34,5 @@
       <parent link="${prefix}world_interface" />
       <child link="${prefix}base_link" />
-      <origin xyz="1.2 3.5 1.65" rpy="0 ${radians(90)} -${radians(90)}" />
+      <origin xyz="1.6 2.8 0.91" rpy="0 0 ${radians(180)}" />
     </joint>
     <joint name="${prefix}joint_1" type="fixed">
