Commit message: add fine alignment step to stabilize output pick point

File: gilbreth_support/urdf/break_beam/break_beam.urdf.xacro (robot description, xacro)
@@ -34,10 +34,10 @@
       <parent link="${prefix}world_interface" />
       <child link="${prefix}base_link" />
-      <origin xyz="1.6 2.8 0.91" rpy="0 0 ${radians(180)}" />
+      <origin xyz="1.6 2.7 0.925" rpy="0 0 ${radians(180)}" />
     </joint>
     <joint name="${prefix}joint_1" type="fixed">
       <parent link="${prefix}base_link" />
       <child link="${prefix}optical_link" />
-      <origin xyz="0 0 0.025" rpy="0 0 0" />
+      <origin xyz="0.025 0 0" rpy="0 0 0" />
     </joint>
   </xacro:macro>
