Commit message: Added conveyor SDF with OSRF gear plugin; added auto-populating parts SDF models and plugin

File: gilbreth_support/urdf/bin/bin.urdf.xacro (robot description, xacro)
@@ -13,5 +13,5 @@
         <origin xyz="0 0 0" rpy="0 0 0"/>
         <geometry>
-          <mesh filename="package://gilbreth_support/meshes/bin/collision/bin_sides.ply"/>
+          <mesh filename="package://gilbreth_support/meshes/bin/collision/bin_sides.dae"/>
         </geometry>
       </collision>
@@ -19,5 +19,5 @@
         <origin xyz="0 0 0" rpy="0 0 0"/>
         <geometry>
-          <mesh filename="package://gilbreth_support/meshes/bin/collision/bin_bottom.ply"/>
+          <mesh filename="package://gilbreth_support/meshes/bin/collision/bin_bottom.dae"/>
         </geometry>
       </collision>
@@ -30,5 +30,13 @@
       </inertial>
     </link>
-    <link name="${prefix}drop_point"/>
+    <link name="${prefix}drop_point">
+      <inertial>
+        <origin xyz="0 0 0" rpy="0 0 0" />
+        <inertia ixx="1.0" ixy="0" ixz="0"
+                 iyy="1.0" iyz="0"
+                 izz="1.0" />
+        <mass value="1.0" />
+      </inertial>
+    </link>
     <!-- joint list -->
     <joint name="${prefix}joint_1" type="fixed">

File: gilbreth_support/urdf/depth_camera/depth_camera.gazebo.xacro (robot description, xacro)
@@ -6,5 +6,5 @@
       <material>Gazebo/Grey</material>
     </gazebo>
-    <gazebo reference="${prefix}focal_point">
+    <gazebo reference="${prefix}camera_link">
       <material>Gazebo/Grey</material>
       <sensor type="depth" name="${camera_name}">
@@ -23,15 +23,11 @@
         </camera>
         <plugin name="${prefix}_controller" filename="libgazebo_ros_openni_kinect.so">
-          <baseline>0.2</baseline>
+          <cameraName>${camera_name}</cameraName>
           <alwaysOn>true</alwaysOn>
           <updateRate>1.0</updateRate>
-          <cameraName>${camera_name}</cameraName>
-          <imageTopicName>/${camera_name}/depth/image_raw</imageTopicName>
-          <cameraInfoTopicName>/${camera_name}/depth/camera_info</cameraInfoTopicName>
-          <depthImageTopicName>/${camera_name}/depth/image_raw</depthImageTopicName>
-          <depthImageInfoTopicName>/${camera_name}/depth/camera_info</depthImageInfoTopicName>
-          <pointCloudTopicName>/${camera_name}/depth/points</pointCloudTopicName>
-          <frameName>${prefix}focal_point</frameName>
           <pointCloudCutoff>0.5</pointCloudCutoff>
+          <baseline>0.2</baseline>
+          <focalLength>0</focalLength>
+          <hackBaseline>0</hackBaseline>
           <distortionK1>0.00000001</distortionK1>
           <distortionK2>0.00000001</distortionK2>
@@ -42,6 +38,10 @@
           <Cx>0</Cx>
           <Cy>0</Cy>
-          <focalLength>0</focalLength>
-          <hackBaseline>0</hackBaseline>
+          <imageTopicName>/${camera_name}/depth/image_raw</imageTopicName>
+          <cameraInfoTopicName>/${camera_name}/depth/camera_info</cameraInfoTopicName>
+          <depthImageTopicName>/${camera_name}/depth/image_raw</depthImageTopicName>
+          <depthImageInfoTopicName>/${camera_name}/depth/camera_info</depthImageInfoTopicName>
+          <pointCloudTopicName>/${camera_name}/depth/points</pointCloudTopicName>
+          <frameName>${prefix}camera_link_optical</frameName>
         </plugin>
       </sensor>

File: gilbreth_support/urdf/depth_camera/depth_camera.urdf.xacro (robot description, xacro)
@@ -31,10 +31,32 @@
       </inertial>
     </link>
-    <link name="${prefix}focal_point"/>
+    <link name="${prefix}camera_link">
+      <inertial>
+        <origin xyz="0 0 0" rpy="0 0 0" />
+        <inertia ixx="0.1" ixy="0" ixz="0"
+                 iyy="0.1" iyz="0"
+                 izz="0.1" />
+        <mass value="1" />
+      </inertial>
+    </link>
+    <link name="${prefix}camera_link_optical">
+      <inertial>
+        <origin xyz="0 0 0" rpy="0 0 0" />
+        <inertia ixx="0.1" ixy="0" ixz="0"
+                 iyy="0.1" iyz="0"
+                 izz="0.1" />
+        <mass value="1" />
+      </inertial>
+    </link>
     <!-- joint list -->
     <joint name="${prefix}joint_1" type="fixed">
       <parent link="${prefix}base_link" />
-      <child link="${prefix}focal_point" />
+      <child link="${prefix}camera_link" />
       <origin xyz="${width / 2} 0 ${height / 2}" rpy="0 0 0" />
+    </joint>
+    <joint name="${prefix}joint_2" type="fixed">
+      <parent link="${prefix}camera_link" />
+      <child link="${prefix}camera_link_optical" />
+      <origin xyz="0 0 0" rpy="-${radians(90)} 0 -${radians(90)}" />
     </joint>
   </xacro:macro>

File: gilbreth_support/urdf/gilbreth.xacro (robot description, xacro)
@@ -1,4 +1,7 @@
 <?xml version="1.0" ?>
 <robot name="gilbreth" xmlns:xacro="http://www.ros.org/wiki/xacro">
+  <!-- linear arm actuator -->
+  <xacro:include filename="$(find gilbreth_support)/urdf/linear_actuator/linear_actuator.xacro" />
+  <xacro:linear_actuator prefix="linear_actuator_"/>
   <!-- include the robot xacro -->
   <xacro:include filename="$(find ur_description)/urdf/ur10.urdf.xacro" />
@@ -8,7 +11,4 @@
   <xacro:include filename="$(find gilbreth_support)/urdf/vacuum_gripper/vacuum_gripper.xacro"/>
   <xacro:vacuum_gripper prefix="vacuum_gripper_"/>
-  <!-- linear arm actuator -->
-  <xacro:include filename="$(find gilbreth_support)/urdf/linear_actuator/linear_actuator.xacro" />
-  <xacro:linear_actuator prefix="linear_actuator_"/>
   <!-- bins -->
   <xacro:include filename="$(find gilbreth_support)/urdf/bin/bin.xacro"/>
@@ -19,7 +19,10 @@
   <xacro:include filename="$(find gilbreth_support)/urdf/depth_camera/depth_camera.xacro"/>
   <xacro:depth_camera prefix="rgbd_1_"/>
+  <!-- break beam -->
+  <xacro:include filename="$(find gilbreth_support)/urdf/break_beam/break_beam.xacro"/>
+  <xacro:break_beam prefix="break_beam_"/>
   <!-- Links -->
   <link name="world"/>
-  <link name="test_link">
+  <link name="workcell">
     <visual>
       <geometry>
@@ -29,5 +32,5 @@
     <collision>
       <geometry>
-        <mesh filename="package://gilbreth_support/meshes/workcell/collision/workcell.ply"/>
+        <mesh filename="package://gilbreth_support/meshes/workcell/collision/workcell.dae"/>
       </geometry>
     </collision>
@@ -39,28 +42,18 @@
     </inertial>
   </link>
-  <link name="conveyor_dummy_link"/>
-  <link name="break_beam" />
   <!-- Joints -->
-  <joint name="test_joint" type="fixed">
+  <joint name="workcell_to_world" type="fixed">
     <parent link="world" />
-    <child link="test_link" />
-    <dynamics friction="1000" damping="1.0"/>
+    <child link="workcell" />
+    <origin xyz="0 0 0" rpy="0 0 ${radians(90)}" />
   </joint>
-  <joint name="conveyor_dummy_to_world" type="fixed">
-    <parent link="test_link" />
-    <child link="conveyor_dummy_link" />
-    <origin xyz="0 -1.2 0.9" rpy="0 0 -${radians(90)}" />
-    <dynamics friction="1000" damping="1.0"/>
-  </joint>
-  <joint name="conveyor_dummy_to_linear_actuator" type="fixed">
-    <parent link="conveyor_dummy_link" />
+  <joint name="linear_actuator_to_workcell" type="fixed">
+    <parent link="world" />
     <child link="linear_actuator_base_link" />
-    <origin xyz="-0.8 0 0" rpy="0 0 0" />
-    <dynamics friction="1000" damping="1.0"/>
+    <origin xyz="0.4 0.0 0.9" rpy="0 0 0" />
   </joint>
   <joint name="robot_to_actuator_carriage" type="fixed">
     <parent link="linear_actuator_carriage" />
     <child link="robot_base_link" />
-    <dynamics friction="5000" damping="1.0"/>
   </joint>
   <joint name="vacuum_gripper_to_robot" type="fixed">
@@ -70,13 +63,13 @@
   <!-- a break_beam type sensor in the frame break_beam_frame -->
   <joint name="break_beam_joint" type="fixed">
-    <parent link="conveyor_dummy_link" />
-    <child link="break_beam" />
-    <origin xyz="0.0 3.5 0.75" rpy="0 0 ${pi}" />
+    <parent link="world" />
+    <child link="break_beam_base_link" />
+    <origin xyz="1.2 3.5 1.65" rpy="0 ${radians(90)} -${radians(90)}" />
   </joint>
   <!-- a kinect camera in the frame kinect_camera_frame -->
   <joint name="camera_link" type="fixed">
-    <parent link="conveyor_dummy_link"/>
+    <parent link="world"/>
     <child link="rgbd_1_base_link" />
-    <origin xyz="0.0 3.0 0.75" rpy="${pi/2} ${pi/2} 0" />
+    <origin xyz="1.2 3.0 1.65" rpy="${radians(90)} ${radians(90)} 0" />
   </joint>
   <!-- a bin in the frame bin1_frame -->

File: gilbreth_support/urdf/linear_actuator/linear_actuator.gazebo.xacro (robot description, xacro)
@@ -8,7 +8,7 @@
       <material>Gazebo/Grey</material>
     </gazebo>
-    <gazebo reference="${prefix}carriage_joint">
+<!--    <gazebo reference="${prefix}carriage_joint">
       <implicitSpringDamper>1</implicitSpringDamper>
-    </gazebo>
+    </gazebo>-->
     <transmission name="${prefix}transmission">
       <type>transmission_interface/SimpleTransmission</type>

File: gilbreth_support/urdf/linear_actuator/linear_actuator.urdf.xacro (robot description, xacro)
@@ -32,5 +32,13 @@
       </inertial>
     </link>
-    <link name="${prefix}carriage"/>
+    <link name="${prefix}carriage">
+      <inertial>
+        <origin xyz="0 0 0" rpy="0 0 0" />
+        <inertia ixx="0.1" ixy="0" ixz="0"
+                 iyy="0.1" iyz="0"
+                 izz="0.1" />
+        <mass value="1" />
+      </inertial>
+    </link>
     <!-- joint list -->
     <joint name="${prefix}carriage_joint" type="prismatic">

File: gilbreth_support/urdf/vacuum_gripper/vacuum_gripper.urdf.xacro (robot description, xacro)
@@ -16,5 +16,5 @@
         <origin xyz="0 0 0" rpy="0 0 0"/>
         <geometry>
-          <mesh filename="package://gilbreth_support/meshes/vacuum_gripper/collision/vacuum_gripper.ply"/>
+          <mesh filename="package://gilbreth_support/meshes/vacuum_gripper/collision/vacuum_gripper.dae"/>
         </geometry>
         <material name="red"/>
@@ -28,5 +28,13 @@
       </inertial>
     </link>
-    <link name="${prefix}tool0"/>
+    <link name="${prefix}tool0">
+      <inertial>
+        <origin xyz="0 0 0" rpy="0 0 0" />
+        <inertia ixx="0.1" ixy="0" ixz="0"
+                 iyy="0.1" iyz="0"
+                 izz="0.1" />
+        <mass value="1" />
+      </inertial>
+    </link>
     <!-- joint list -->
     <joint name="vacuum_gripper_joint" type="fixed">

Commit message: added a bin
fixed model_path bug

rescaled bin size

added a new bin

changed rostopic

modified for debugging

new package dependencies

new package dependencies

defined new traj. msg

defined new msg

added new bin

added grasp planning functionality

added new bin

launch rviz

tuned parameters

added new bins

nothing changed

demo scripts

grasp planning functionality

rospy setup file

tuned some parameters

added new dependency

Demo description

deleted

File: gilbreth_support/urdf/bin/bin.urdf.xacro (robot description, xacro)
@@ -8,4 +8,5 @@
         <geometry>
           <mesh filename="package://gilbreth_support/meshes/bin/visual/bin.dae" />
+          <scale>0.6 0.6 0.6</scale>
         </geometry>
       </visual>
@@ -14,4 +15,5 @@
         <geometry>
           <mesh filename="package://gilbreth_support/meshes/bin/collision/bin_bottom.dae"/>
+          <scale>0.6 0.6 0.6</scale>
         </geometry>
       </collision>
@@ -20,4 +22,5 @@
         <geometry>
           <mesh filename="package://gilbreth_support/meshes/bin/collision/bin_sides.dae"/>
+          <scale>0.6 0.6 0.6</scale>
         </geometry>
       </collision>

File: gilbreth_support/urdf/gilbreth.xacro (robot description, xacro)
@@ -8,4 +8,6 @@
   <xacro:bin_urdf prefix="bin_2_"/>
   <xacro:bin_urdf prefix="bin_3_"/>
+  <xacro:bin_urdf prefix="bin_4_"/>
+  <xacro:bin_urdf prefix="bin_5_"/>
   <!-- depth camera -->
   <xacro:include filename="$(find gilbreth_support)/urdf/depth_camera/depth_camera.urdf.xacro"/>
@@ -35,5 +37,5 @@
     <parent link="world" />
     <child link="bin_1_base_link" />
-    <origin xyz="-0.4 -1.0 0.0" rpy="0 0 0" />
+    <origin xyz="-0.3 -1.2 0.0" rpy="0 0 0" />
   </joint>
   <!-- a bin in the frame bin2_frame -->
@@ -41,5 +43,5 @@
     <parent link="world" />
     <child link="bin_2_base_link" />
-    <origin xyz="-0.4 0.0 0.0" rpy="0 0 0" />
+    <origin xyz="-0.3 -0.4 0.0" rpy="0 0 0" />
   </joint>
   <!-- a bin in the frame bin3_frame -->
@@ -47,5 +49,17 @@
     <parent link="world" />
     <child link="bin_3_base_link" />
-    <origin xyz="-0.4 1.0 0.0" rpy="0 0 0" />
+    <origin xyz="-0.3 0.4 0.0" rpy="0 0 0" />
+  </joint>
+  <!-- a bin in the frame bin4_frame -->
+  <joint name="bin_4_joint" type="fixed">
+    <parent link="world" />
+    <child link="bin_4_base_link" />
+    <origin xyz="-0.3 1.2 0.0" rpy="0 0 0" />
+  </joint>
+  <!-- a bin in the frame bin5_frame -->
+  <joint name="bin_5_joint" type="fixed">
+    <parent link="world" />
+    <child link="bin_5_base_link" />
+    <origin xyz="-0.3 -2.0 0.0" rpy="0 0 0" />
   </joint>
 </robot>
