Commit message: Modified urdf files so that the xacro properties and included macros are private within the macro; moved some plugin functionality from gazebo urdf files to gazebo world

File: gilbreth_support/urdf/bin/bin.gazebo.xacro (robot description, xacro)
@@ -8,12 +8,15 @@
           <collision>${prefix}bin_contact</collision>
         </contact>
-        <plugin name="${prefix}object_disposal_plugin" filename="libObjectDisposalPlugin.so">
-          <contact_sensor_name>object_disposal_contact</contact_sensor_name>
-          <center_of_gravity_check>true</center_of_gravity_check>
-          <robot_namespace>/gilbreth</robot_namespace>
-          <control_topic>object_disposal/control</control_topic>
-          <state_topic>object_disposal/state</state_topic>
-        </plugin>
       </sensor>
+    </gazebo>
+    <gazebo>
+      <static>true</static>
+      <plugin name="${prefix}object_disposal_plugin" filename="libObjectDisposalPlugin.so">
+        <contact_sensor_name>${prefix}contact_sensor</contact_sensor_name>
+<!--        <contact_side_normal>1 0 0</contact_side_normal>-->
+        <center_of_gravity_check>true</center_of_gravity_check>
+        <disposal_pose>30 30 0 0 0 0</disposal_pose>
+        <update_rate>5</update_rate>
+      </plugin>
     </gazebo>
   </xacro:macro>

File: gilbreth_support/urdf/bin/bin.xacro (robot description, xacro)
@@ -1,11 +1,10 @@
 <?xml version="1.0"?>
 <robot name="bin" xmlns:xacro="http://www.ros.org/wiki/xacro">
-  <xacro:macro name="bin" params="prefix">
-    <!-- URDF -->
-    <xacro:include filename="$(find gilbreth_support)/urdf/bin/bin.urdf.xacro"/>
-    <xacro:bin_urdf prefix="${prefix}"/>
-    <!-- Gazebo -->
-    <xacro:include filename="$(find gilbreth_support)/urdf/bin/bin.gazebo.xacro"/>
-    <xacro:bin_gazebo prefix="${prefix}"/>
-  </xacro:macro>
+  <arg name="prefix" default="bin_"/>
+  <!-- URDF -->
+  <xacro:include filename="$(find gilbreth_support)/urdf/bin/bin.urdf.xacro"/>
+  <xacro:bin_urdf prefix="$(arg prefix)"/>
+  <!-- Gazebo -->
+  <xacro:include filename="$(find gilbreth_support)/urdf/bin/bin.gazebo.xacro"/>
+  <xacro:bin_gazebo prefix="$(arg prefix)"/>
 </robot>

File: gilbreth_support/urdf/break_beam/break_beam.gazebo.xacro (robot description, xacro)
@@ -33,9 +33,12 @@
         <always_on>1</always_on>
         <plugin name="${prefix}controller" filename="libgazebo_ros_laser.so" >
-          <topicName>/gilbreth/laser/scan</topicName>
+          <topicName>laser/scan</topicName>
           <frameName>${prefix}optical_link</frameName>
         </plugin>
       </sensor>
     </gazebo>
+    <gazebo>
+      <static>true</static>
+    </gazebo>
   </xacro:macro>
 </robot>

File: gilbreth_support/urdf/break_beam/break_beam.urdf.xacro (robot description, xacro)
@@ -3,4 +3,5 @@
   <xacro:macro name="break_beam_urdf" params="prefix">
     <!-- link list -->
+    <link name="${prefix}world_interface"/>
     <link name="${prefix}base_link">
       <visual>
@@ -28,14 +29,11 @@
       </inertial>
     </link>
-    <link name="${prefix}optical_link">
-      <inertial>
-        <origin xyz="0 0 0" rpy="0 0 0" />
-        <inertia ixx="0.1" ixy="0" ixz="0"
-                 iyy="0.1" iyz="0"
-                 izz="0.1" />
-        <mass value="1" />
-      </inertial>
-    </link>
+    <link name="${prefix}optical_link"/>
     <!-- joint list -->
+    <joint name="${prefix}world_joint" type="fixed">
+      <parent link="${prefix}world_interface" />
+      <child link="${prefix}base_link" />
+      <origin xyz="1.2 3.5 1.65" rpy="0 ${radians(90)} -${radians(90)}" />
+    </joint>
     <joint name="${prefix}joint_1" type="fixed">
       <parent link="${prefix}base_link" />

File: gilbreth_support/urdf/break_beam/break_beam.xacro (robot description, xacro)
@@ -1,11 +1,10 @@
 <?xml version="1.0"?>
 <robot name="break_beam" xmlns:xacro="http://www.ros.org/wiki/xacro">
-  <xacro:macro name="break_beam" params="prefix">
-    <!-- URDF -->
-    <xacro:include filename="$(find gilbreth_support)/urdf/break_beam/break_beam.urdf.xacro"/>
-    <xacro:break_beam_urdf prefix="${prefix}"/>
-    <!-- Gazebo -->
-    <xacro:include filename="$(find gilbreth_support)/urdf/break_beam/break_beam.gazebo.xacro"/>
-    <xacro:break_beam_gazebo prefix="${prefix}"/>
-  </xacro:macro>
+  <arg name="prefix" default="break_beam_"/>
+  <!-- URDF -->
+  <xacro:include filename="$(find gilbreth_support)/urdf/break_beam/break_beam.urdf.xacro"/>
+  <xacro:break_beam_urdf prefix="$(arg prefix)"/>
+  <!-- Gazebo -->
+  <xacro:include filename="$(find gilbreth_support)/urdf/break_beam/break_beam.gazebo.xacro"/>
+  <xacro:break_beam_gazebo prefix="$(arg prefix)"/>
 </robot>

File: gilbreth_support/urdf/depth_camera/depth_camera.gazebo.xacro (robot description, xacro)
@@ -2,5 +2,5 @@
 <robot name="depth_camera_gazebo" xmlns:xacro="http://www.ros.org/wiki/xacro">
   <xacro:macro name="depth_camera_gazebo" params="prefix">
-    <xacro:property name="camera_name" value="${prefix}sensor"/>
+    <xacro:property name="camera_name" value="${prefix}"/>
     <gazebo reference="${prefix}base_link">
       <material>Gazebo/Grey</material>
@@ -24,4 +24,5 @@
         <plugin name="${prefix}_controller" filename="libgazebo_ros_openni_kinect.so">
           <cameraName>${camera_name}</cameraName>
+          <frameName>${prefix}camera_link_optical</frameName>
           <alwaysOn>true</alwaysOn>
           <updateRate>1.0</updateRate>
@@ -38,13 +39,15 @@
           <Cx>0</Cx>
           <Cy>0</Cy>
-          <imageTopicName>/${camera_name}/depth/image_raw</imageTopicName>
-          <cameraInfoTopicName>/${camera_name}/depth/camera_info</cameraInfoTopicName>
-          <depthImageTopicName>/${camera_name}/depth/image_raw</depthImageTopicName>
-          <depthImageInfoTopicName>/${camera_name}/depth/camera_info</depthImageInfoTopicName>
-          <pointCloudTopicName>/${camera_name}/depth/points</pointCloudTopicName>
-          <frameName>${prefix}camera_link_optical</frameName>
+          <imageTopicName>${camera_name}/depth/image_raw</imageTopicName>
+          <cameraInfoTopicName>${camera_name}/depth/camera_info</cameraInfoTopicName>
+          <depthImageTopicName>${camera_name}/depth/image_raw</depthImageTopicName>
+          <depthImageInfoTopicName>${camera_name}/depth/camera_info</depthImageInfoTopicName>
+          <pointCloudTopicName>${camera_name}/depth/points</pointCloudTopicName>
         </plugin>
       </sensor>
     </gazebo>
+    <gazebo>
+      <static>true</static>
+    </gazebo>
   </xacro:macro>
 </robot>

File: gilbreth_support/urdf/depth_camera/depth_camera.urdf.xacro (robot description, xacro)
@@ -1,9 +1,10 @@
 <?xml version="1.0"?>
 <robot name="depth_camera_urdf" xmlns:xacro="http://www.ros.org/wiki/xacro">
-  <xacro:property name="length" value="0.2"/>
-  <xacro:property name="width" value="0.050"/>
-  <xacro:property name="height" value="0.050"/>
   <xacro:macro name="depth_camera_urdf" params="prefix">
+    <xacro:property name="length" value="0.2"/>
+    <xacro:property name="width" value="0.050"/>
+    <xacro:property name="height" value="0.050"/>
     <!-- link list -->
+    <link name="${prefix}world_interface"/>
     <link name="${prefix}base_link">
       <visual>
@@ -31,29 +32,18 @@
       </inertial>
     </link>
-    <link name="${prefix}camera_link">
-      <inertial>
-        <origin xyz="0 0 0" rpy="0 0 0" />
-        <inertia ixx="0.1" ixy="0" ixz="0"
-                 iyy="0.1" iyz="0"
-                 izz="0.1" />
-        <mass value="1" />
-      </inertial>
-    </link>
-    <link name="${prefix}camera_link_optical">
-      <inertial>
-        <origin xyz="0 0 0" rpy="0 0 0" />
-        <inertia ixx="0.1" ixy="0" ixz="0"
-                 iyy="0.1" iyz="0"
-                 izz="0.1" />
-        <mass value="1" />
-      </inertial>
-    </link>
+    <link name="${prefix}camera_link"/>
+    <link name="${prefix}camera_link_optical"/>
     <!-- joint list -->
     <joint name="${prefix}joint_1" type="fixed">
+      <parent link="${prefix}world_interface" />
+      <child link="${prefix}base_link" />
+      <origin xyz="1.2 3.0 1.65" rpy="0 ${radians(90)} -${radians(90)}" />
+    </joint>
+    <joint name="${prefix}joint_2" type="fixed">
       <parent link="${prefix}base_link" />
       <child link="${prefix}camera_link" />
       <origin xyz="${width / 2} 0 ${height / 2}" rpy="0 0 0" />
     </joint>
-    <joint name="${prefix}joint_2" type="fixed">
+    <joint name="${prefix}joint_3" type="fixed">
       <parent link="${prefix}camera_link" />
       <child link="${prefix}camera_link_optical" />

File: gilbreth_support/urdf/depth_camera/depth_camera.xacro (robot description, xacro)
@@ -1,11 +1,10 @@
 <?xml version="1.0"?>
 <robot name="depth_camera" xmlns:xacro="http://www.ros.org/wiki/xacro">
-  <xacro:macro name="depth_camera" params="prefix">
-    <!-- URDF -->
-    <xacro:include filename="$(find gilbreth_support)/urdf/depth_camera/depth_camera.urdf.xacro"/>
-    <xacro:depth_camera_urdf prefix="${prefix}"/>
-    <!-- Gazebo -->
-    <xacro:include filename="$(find gilbreth_support)/urdf/depth_camera/depth_camera.gazebo.xacro"/>
-    <xacro:depth_camera_gazebo prefix="${prefix}"/>
-  </xacro:macro>
+  <arg name="prefix" default="depth_camera_"/>
+  <!-- URDF -->
+  <xacro:include filename="$(find gilbreth_support)/urdf/depth_camera/depth_camera.urdf.xacro"/>
+  <xacro:depth_camera_urdf prefix="$(arg prefix)"/>
+  <!-- Gazebo -->
+  <xacro:include filename="$(find gilbreth_support)/urdf/depth_camera/depth_camera.gazebo.xacro"/>
+  <xacro:depth_camera_gazebo prefix="$(arg prefix)"/>
 </robot>

File: gilbreth_support/urdf/gilbreth.xacro (robot description, xacro)
@@ -2,55 +2,34 @@
 <robot name="gilbreth" xmlns:xacro="http://www.ros.org/wiki/xacro">
   <!-- linear arm actuator -->
-  <xacro:include filename="$(find gilbreth_support)/urdf/linear_actuator/linear_actuator.xacro" />
-  <xacro:linear_actuator prefix="linear_actuator_"/>
+  <xacro:include filename="$(find gilbreth_support)/urdf/linear_actuator/linear_actuator.urdf.xacro" />
+  <xacro:linear_actuator_urdf prefix="linear_actuator_"/>
   <!-- include the robot xacro -->
-  <xacro:include filename="$(find ur_description)/urdf/ur10.urdf.xacro" />
-  <xacro:ur10_robot prefix="robot_" joint_limited="false"/>
+<!--  <xacro:include filename="$(find ur_description)/urdf/ur10.urdf.xacro" />
+  <xacro:ur10_robot prefix="robot_" joint_limited="false"/>-->
   <!-- vacuum gripper -->
-  <xacro:property name="vacuum_gripper" value="vacuum_gripper_" />
-  <xacro:include filename="$(find gilbreth_support)/urdf/vacuum_gripper/vacuum_gripper.xacro"/>
-  <xacro:vacuum_gripper prefix="vacuum_gripper_"/>
+<!--  <xacro:include filename="$(find gilbreth_support)/urdf/vacuum_gripper/vacuum_gripper.urdf.xacro"/>
+  <xacro:vacuum_gripper_urdf prefix="vacuum_gripper_"/>-->
   <!-- bins -->
-  <xacro:include filename="$(find gilbreth_support)/urdf/bin/bin.xacro"/>
+<!--  <xacro:include filename="$(find gilbreth_support)/urdf/bin/bin.xacro"/>
   <xacro:bin prefix="bin_1_"/>
   <xacro:bin prefix="bin_2_"/>
-  <xacro:bin prefix="bin_3_"/>
+  <xacro:bin prefix="bin_3_"/>-->
   <!-- depth camera -->
-  <xacro:include filename="$(find gilbreth_support)/urdf/depth_camera/depth_camera.xacro"/>
-  <xacro:depth_camera prefix="rgbd_1_"/>
+  <xacro:include filename="$(find gilbreth_support)/urdf/depth_camera/depth_camera.urdf.xacro"/>
+  <xacro:depth_camera_urdf prefix="depth_camera_"/>
   <!-- break beam -->
-  <xacro:include filename="$(find gilbreth_support)/urdf/break_beam/break_beam.xacro"/>
-  <xacro:break_beam prefix="break_beam_"/>
-  <!-- Links -->
-  <link name="world"/>
-  <link name="workcell">
-    <visual>
-      <geometry>
-        <mesh filename="package://gilbreth_support/meshes/workcell/visual/workcell.dae"/>
-      </geometry>
-    </visual>
-    <collision>
-      <geometry>
-        <mesh filename="package://gilbreth_support/meshes/workcell/collision/workcell.dae"/>
-      </geometry>
-    </collision>
-    <inertial>
-      <inertia ixx="1.0" ixy="0" ixz="0"
-               iyy="1.0" iyz="0"
-               izz="1.0" />
-      <mass value="100" />
-    </inertial>
-  </link>
+  <xacro:include filename="$(find gilbreth_support)/urdf/break_beam/break_beam.urdf.xacro"/>
+  <xacro:break_beam_urdf prefix="break_beam_"/>
+  <!-- workcell -->
+  <xacro:include filename="$(find gilbreth_support)/urdf/workcell/workcell.xacro"/>
   <!-- Joints -->
   <joint name="workcell_to_world" type="fixed">
     <parent link="world" />
-    <child link="workcell" />
-    <origin xyz="0 0 0" rpy="0 0 ${radians(90)}" />
+    <child link="world_interface" />
   </joint>
-  <joint name="linear_actuator_to_workcell" type="fixed">
+<!--  <joint name="linear_actuator_to_workcell" type="fixed">
     <parent link="world" />
-    <child link="linear_actuator_base_link" />
-    <origin xyz="0.4 0.0 0.9" rpy="0 0 0" />
-  </joint>
+    <child link="linear_actuator_world_interface" />
+  </joint>-->
   <joint name="robot_to_actuator_carriage" type="fixed">
     <parent link="linear_actuator_carriage" />
@@ -64,35 +43,28 @@
   <joint name="break_beam_joint" type="fixed">
     <parent link="world" />
-    <child link="break_beam_base_link" />
-    <origin xyz="1.2 3.5 1.65" rpy="0 ${radians(90)} -${radians(90)}" />
+    <child link="break_beam_world_interface" />
   </joint>
   <!-- a kinect camera in the frame kinect_camera_frame -->
   <joint name="camera_link" type="fixed">
     <parent link="world"/>
-    <child link="rgbd_1_base_link" />
-    <origin xyz="1.2 3.0 1.65" rpy="${radians(90)} ${radians(90)} 0" />
+    <child link="depth_camera_world_interface" />
   </joint>
   <!-- a bin in the frame bin1_frame -->
-  <joint name="bin_1_joint" type="fixed">
+<!--  <joint name="bin_1_joint" type="fixed">
     <parent link="linear_actuator_base_link" />
     <child link="bin_1_base_link" />
     <origin xyz="-0.8 -1.0 -0.9" rpy="0 0 0" />
-  </joint>
+  </joint>-->
   <!-- a bin in the frame bin2_frame -->
-  <joint name="bin_2_joint" type="fixed">
+<!--  <joint name="bin_2_joint" type="fixed">
     <parent link="linear_actuator_base_link" />
     <child link="bin_2_base_link" />
     <origin xyz="-0.8 0.0 -0.9" rpy="0 0 0" />
-  </joint>
+  </joint>-->
   <!-- a bin in the frame bin3_frame -->
-  <joint name="bin_3_joint" type="fixed">
+<!--  <joint name="bin_3_joint" type="fixed">
     <parent link="linear_actuator_base_link" />
     <child link="bin_3_base_link" />
     <origin xyz="-0.8 1.0 -0.9" rpy="0 0 0" />
-  </joint>
-  <gazebo>
-    <plugin name="gazebo_ros_control" filename="libgazebo_ros_control.so">
-      <robotNamespace>/</robotNamespace>
-    </plugin>
-  </gazebo>
+  </joint>-->
 </robot>

File: gilbreth_support/urdf/linear_actuator/linear_actuator.gazebo.xacro (robot description, xacro)
@@ -20,4 +20,11 @@
       </actuator>
     </transmission>
+    <gazebo>
+<!--      <static>true</static>-->
+      <plugin name="gazebo_ros_control" filename="libgazebo_ros_control.so">
+        <robotNamespace>gilbreth</robotNamespace>
+        <robotParam>${prefix}description</robotParam>
+      </plugin>
+    </gazebo>
   </xacro:macro>
 </robot>

File: gilbreth_support/urdf/linear_actuator/linear_actuator.urdf.xacro (robot description, xacro)
@@ -1,10 +1,15 @@
 <?xml version="1.0"?>
 <robot name="linear_actuator_urdf" xmlns:xacro="http://www.ros.org/wiki/xacro">
-  <xacro:property name="width" value="0.2" />
-  <xacro:property name="length" value="4.6" />
-  <xacro:property name="height" value="0.1" />
-  <xacro:property name="carriage_length" value="0.2"/>
   <xacro:macro name="linear_actuator_urdf" params="prefix">
+    <xacro:property name="width" value="0.2" />
+    <xacro:property name="length" value="4.6" />
+    <xacro:property name="height" value="0.1" />
+    <xacro:property name="carriage_length" value="0.2"/>
+    <xacro:include filename="$(find ur_description)/urdf/ur10.urdf.xacro"/>
+    <xacro:ur10_robot prefix="robot_" joint_limited="false"/>
+    <xacro:include filename="$(find gilbreth_support)/urdf/vacuum_gripper/vacuum_gripper.urdf.xacro"/>
+    <xacro:vacuum_gripper_urdf prefix="vacuum_gripper_"/>
     <!-- link list -->
+    <link name="world"/>
     <link name="${prefix}base_link">
       <visual>
@@ -42,4 +47,9 @@
     </link>
     <!-- joint list -->
+    <joint name="${prefix}world_joint" type="fixed">
+      <parent link="world" />
+      <child link="${prefix}base_link" />
+      <origin xyz="0.4 0.0 0.9" rpy="0 0 0" />
+    </joint>
     <joint name="${prefix}carriage_joint" type="prismatic">
       <parent link="${prefix}base_link" />
@@ -53,4 +63,12 @@
       <dynamics damping="0.7" friction="500.0" />
     </joint>
+    <joint name="${prefix}joint_2" type="fixed">
+      <parent link="${prefix}carriage" />
+      <child link="robot_base_link" />
+    </joint>
+    <joint name="${prefix}joint_3" type="fixed">
+      <parent link="robot_tool0" />
+      <child link="vacuum_gripper_base_link" />
+    </joint>
   </xacro:macro>
 </robot>

File: gilbreth_support/urdf/linear_actuator/linear_actuator.xacro (robot description, xacro)
@@ -1,11 +1,10 @@
 <?xml version="1.0"?>
 <robot name="linear_actuator" xmlns:xacro="http://www.ros.org/wiki/xacro">
-  <xacro:macro name="linear_actuator" params="prefix">
-    <!-- URDF -->
-    <xacro:include filename="$(find gilbreth_support)/urdf/linear_actuator/linear_actuator.urdf.xacro"/>
-    <xacro:linear_actuator_urdf prefix="${prefix}"/>
-    <!-- Gazebo -->
-    <xacro:include filename="$(find gilbreth_support)/urdf/linear_actuator/linear_actuator.gazebo.xacro"/>
-    <xacro:linear_actuator_gazebo prefix="${prefix}" joint_interface="hardware_interface/PositionJointInterface"/>
-  </xacro:macro>
+  <arg name="prefix" default="linear_actuator_"/>
+  <!-- URDF -->
+  <xacro:include filename="$(find gilbreth_support)/urdf/linear_actuator/linear_actuator.urdf.xacro"/>
+  <xacro:linear_actuator_urdf prefix="$(arg prefix)"/>
+  <!-- Gazebo -->
+  <xacro:include filename="$(find gilbreth_support)/urdf/linear_actuator/linear_actuator.gazebo.xacro"/>
+  <xacro:linear_actuator_gazebo prefix="$(arg prefix)" joint_interface="hardware_interface/PositionJointInterface"/>
 </robot>

File: gilbreth_support/urdf/vacuum_gripper/vacuum_gripper.gazebo.xacro (robot description, xacro)
@@ -16,5 +16,5 @@
         </grasp_check>
         <xacro:insert_block name="drops_info" />
-        <suction_cup_link>${prefix}tool0</suction_cup_link>
+        <suction_cup_link>${prefix}::${prefix}base_link</suction_cup_link>
         <!-- ROS -->
         <robot_namespace>/gilbreth</robot_namespace>

File: gilbreth_support/urdf/vacuum_gripper/vacuum_gripper.urdf.xacro (robot description, xacro)
@@ -29,5 +29,5 @@
     </link>
     <link name="${prefix}tool0">
-      <inertial>
+<!--      <inertial>
         <origin xyz="0 0 0" rpy="0 0 0" />
         <inertia ixx="0.1" ixy="0" ixz="0"
@@ -35,5 +35,5 @@
                  izz="0.1" />
         <mass value="1" />
-      </inertial>
+      </inertial>-->
     </link>
     <!-- joint list -->

File: gilbreth_support/urdf/vacuum_gripper/vacuum_gripper.xacro (robot description, xacro)
@@ -1,13 +1,12 @@
 <?xml version="1.0"?>
 <robot name="vacuum_gripper" xmlns:xacro="http://www.ros.org/wiki/xacro">
-  <xacro:macro name="vacuum_gripper" params="prefix">
-    <!-- URDF -->
-    <xacro:include filename="$(find gilbreth_support)/urdf/vacuum_gripper/vacuum_gripper.urdf.xacro"/>
-    <xacro:vacuum_gripper_urdf prefix="${prefix}"/>
-    <!-- Gazebo -->
-    <xacro:include filename="$(find gilbreth_support)/urdf/vacuum_gripper/vacuum_gripper.gazebo.xacro"/>
-    <xacro:vacuum_gripper_gazebo prefix="${prefix}">
-      <drops_info/>
-    </xacro:vacuum_gripper_gazebo>
-  </xacro:macro>
+  <arg name="prefix" default="vacuum_gripper_"/>
+  <!-- URDF -->
+  <xacro:include filename="$(find gilbreth_support)/urdf/vacuum_gripper/vacuum_gripper.urdf.xacro"/>
+  <xacro:vacuum_gripper_urdf prefix="$(arg prefix)"/>
+  <!-- Gazebo -->
+  <xacro:include filename="$(find gilbreth_support)/urdf/vacuum_gripper/vacuum_gripper.gazebo.xacro"/>
+  <xacro:vacuum_gripper_gazebo prefix="$(arg prefix)">
+    <drops_info/>
+  </xacro:vacuum_gripper_gazebo>
 </robot>
