Commit message: Added bins capable of deleting objects dropped inside of them to the simulation environment

File: gilbreth_support/urdf/bin/bin.gazebo.xacro (robot description, xacro)
@@ -6,5 +6,5 @@
         <update_rate>10</update_rate>
         <contact>
-          <collision>${prefix}bin_contact</collision>
+          <collision>${prefix}base_link_collision</collision>
         </contact>
       </sensor>
@@ -14,8 +14,7 @@
       <plugin name="${prefix}object_disposal_plugin" filename="libObjectDisposalPlugin.so">
         <contact_sensor_name>${prefix}contact_sensor</contact_sensor_name>
-<!--        <contact_side_normal>1 0 0</contact_side_normal>-->
-        <center_of_gravity_check>true</center_of_gravity_check>
-        <disposal_pose>30 30 0 0 0 0</disposal_pose>
-        <update_rate>5</update_rate>
+        <contact_side_normal>0 0 1</contact_side_normal>
+        <disposal_pose>0 0 0 0 0 0</disposal_pose>
+        <update_rate>1</update_rate>
       </plugin>
     </gazebo>

File: gilbreth_support/urdf/bin/bin.urdf.xacro (robot description, xacro)
@@ -13,11 +13,11 @@
         <origin xyz="0 0 0" rpy="0 0 0"/>
         <geometry>
-          <mesh filename="package://gilbreth_support/meshes/bin/collision/bin_sides.dae"/>
+          <mesh filename="package://gilbreth_support/meshes/bin/collision/bin_bottom.dae"/>
         </geometry>
       </collision>
-      <collision name="${prefix}bin_contact">
+      <collision>
         <origin xyz="0 0 0" rpy="0 0 0"/>
         <geometry>
-          <mesh filename="package://gilbreth_support/meshes/bin/collision/bin_bottom.dae"/>
+          <mesh filename="package://gilbreth_support/meshes/bin/collision/bin_sides.dae"/>
         </geometry>
       </collision>

File: gilbreth_support/urdf/bin/bin.xacro (robot description, xacro)
@@ -1,5 +1,5 @@
 <?xml version="1.0"?>
 <robot name="bin" xmlns:xacro="http://www.ros.org/wiki/xacro">
-  <arg name="prefix" default="bin_"/>
+  <arg name="prefix" default="bin_1_"/>
   <!-- URDF -->
   <xacro:include filename="$(find gilbreth_support)/urdf/bin/bin.urdf.xacro"/>

File: gilbreth_support/urdf/gilbreth.xacro (robot description, xacro)
@@ -4,8 +4,8 @@
   <xacro:include filename="$(find gilbreth_support)/urdf/robot_system/robot_system.xacro"/>
   <!-- bins -->
-<!--  <xacro:include filename="$(find gilbreth_support)/urdf/bin/bin.xacro"/>
-  <xacro:bin prefix="bin_1_"/>
-  <xacro:bin prefix="bin_2_"/>
-  <xacro:bin prefix="bin_3_"/>-->
+  <xacro:include filename="$(find gilbreth_support)/urdf/bin/bin.urdf.xacro"/>
+  <xacro:bin_urdf prefix="bin_1_"/>
+  <xacro:bin_urdf prefix="bin_2_"/>
+  <xacro:bin_urdf prefix="bin_3_"/>
   <!-- depth camera -->
   <xacro:include filename="$(find gilbreth_support)/urdf/depth_camera/depth_camera.urdf.xacro"/>
@@ -32,20 +32,20 @@
   </joint>
   <!-- a bin in the frame bin1_frame -->
-<!--  <joint name="bin_1_joint" type="fixed">
-    <parent link="linear_actuator_base_link" />
+  <joint name="bin_1_joint" type="fixed">
+    <parent link="world" />
     <child link="bin_1_base_link" />
-    <origin xyz="-0.8 -1.0 -0.9" rpy="0 0 0" />
-  </joint>-->
+    <origin xyz="-0.4 -1.0 0.0" rpy="0 0 0" />
+  </joint>
   <!-- a bin in the frame bin2_frame -->
-<!--  <joint name="bin_2_joint" type="fixed">
-    <parent link="linear_actuator_base_link" />
+  <joint name="bin_2_joint" type="fixed">
+    <parent link="world" />
     <child link="bin_2_base_link" />
-    <origin xyz="-0.8 0.0 -0.9" rpy="0 0 0" />
-  </joint>-->
+    <origin xyz="-0.4 0.0 0.0" rpy="0 0 0" />
+  </joint>
   <!-- a bin in the frame bin3_frame -->
-<!--  <joint name="bin_3_joint" type="fixed">
-    <parent link="linear_actuator_base_link" />
+  <joint name="bin_3_joint" type="fixed">
+    <parent link="world" />
     <child link="bin_3_base_link" />
-    <origin xyz="-0.8 1.0 -0.9" rpy="0 0 0" />
-  </joint>-->
+    <origin xyz="-0.4 1.0 0.0" rpy="0 0 0" />
+  </joint>
 </robot>

Commit message: new tool and traj planner
added tray models

modified gazebo environment

new gripper

changed params

deleted

slow down conveyor

merge from ll

new params

new tool and traj planner

File: gilbreth_support/urdf/bin/bin.gazebo.xacro (robot description, xacro)
@@ -12,10 +12,10 @@
     <gazebo>
       <static>true</static>
-      <plugin name="${prefix}object_disposal_plugin" filename="libObjectDisposalPlugin.so">
+      <!--plugin name="${prefix}object_disposal_plugin" filename="libObjectDisposalPlugin.so">
         <contact_sensor_name>${prefix}contact_sensor</contact_sensor_name>
         <contact_side_normal>0 0 1</contact_side_normal>
         <disposal_pose>0 0 0 0 0 0</disposal_pose>
         <update_rate>1</update_rate>
-      </plugin>
+      </plugin-->
     </gazebo>
   </xacro:macro>

File: gilbreth_support/urdf/break_beam/break_beam.urdf.xacro (robot description, xacro)
@@ -34,10 +34,10 @@
       <parent link="${prefix}world_interface" />
       <child link="${prefix}base_link" />
-      <origin xyz="1.6 2.8 0.91" rpy="0 0 ${radians(180)}" />
+      <origin xyz="1.6 2.8 0.925" rpy="0 0 ${radians(180)}" />
     </joint>
     <joint name="${prefix}joint_1" type="fixed">
       <parent link="${prefix}base_link" />
       <child link="${prefix}optical_link" />
-      <origin xyz="0 0 0.025" rpy="0 0 0" />
+      <origin xyz="0.025 0 0.0" rpy="0 0 0" />
     </joint>
   </xacro:macro>

File: gilbreth_support/urdf/robot_system/robot_system.xacro (robot description, xacro)
@@ -13,10 +13,17 @@
   <xacro:ur10_robot prefix="${robot_prefix}" joint_limited="true"/>
   <!-- Vacuum Gripper -->
-  <xacro:include filename="$(find gilbreth_support)/urdf/vacuum_gripper/vacuum_gripper.urdf.xacro"/>
+  <!--xacro:include filename="$(find gilbreth_support)/urdf/vacuum_gripper/vacuum_gripper.urdf.xacro"/>
   <xacro:vacuum_gripper_urdf prefix="${vacuum_gripper_prefix}"/>
   <xacro:include filename="$(find gilbreth_support)/urdf/vacuum_gripper/vacuum_gripper.gazebo.xacro"/>
   <xacro:vacuum_gripper_gazebo prefix="${vacuum_gripper_prefix}" gripper_link="robot_system_::robot_wrist_3_link">
     <drops_info/>
-  </xacro:vacuum_gripper_gazebo>
+  </xacro:vacuum_gripper_gazebo-->
+  <!-- Simple Vacuum Gripper -->
+  <xacro:include filename="$(find gilbreth_support)/urdf/simple_gripper/simple_gripper.urdf.xacro"/>
+  <xacro:simple_gripper_urdf prefix="${vacuum_gripper_prefix}"/>
+  <xacro:include filename="$(find gilbreth_support)/urdf/simple_gripper/simple_gripper.gazebo.xacro"/>
+  <xacro:simple_gripper_gazebo prefix="${vacuum_gripper_prefix}" gripper_link="robot_system_::robot_wrist_3_link">
+    <drops_info/>
+  </xacro:simple_gripper_gazebo>
   <!-- Joints -->
   <joint name="robot_to_carriage" type="fixed">
