Commit message: deleted old gripper
modified gripper

modified params

added robot arm controller

modified controller params

a slower velocity param

resolved problems

new execution code

added robot controller

deleted traj node

added test and exec node

Update tool_plan_param.yaml

resolved a mistake

File: gilbreth_support/urdf/robot_system/robot_system.xacro (robot description, xacro)
@@ -12,11 +12,11 @@
   <xacro:include filename="$(find ur_description)/urdf/ur10.urdf.xacro"/>
   <xacro:ur10_robot prefix="${robot_prefix}" joint_limited="true"/>
-  <!-- Vacuum Gripper -->
-  <xacro:include filename="$(find gilbreth_support)/urdf/vacuum_gripper/vacuum_gripper.urdf.xacro"/>
-  <xacro:vacuum_gripper_urdf prefix="${vacuum_gripper_prefix}"/>
-  <xacro:include filename="$(find gilbreth_support)/urdf/vacuum_gripper/vacuum_gripper.gazebo.xacro"/>
-  <xacro:vacuum_gripper_gazebo prefix="${vacuum_gripper_prefix}" gripper_link="robot_system_::robot_wrist_3_link">
+  <!-- Simple Vacuum Gripper -->
+  <xacro:include filename="$(find gilbreth_support)/urdf/simple_gripper/simple_gripper.urdf.xacro"/>
+  <xacro:simple_gripper_urdf prefix="${vacuum_gripper_prefix}"/>
+  <xacro:include filename="$(find gilbreth_support)/urdf/simple_gripper/simple_gripper.gazebo.xacro"/>
+  <xacro:simple_gripper_gazebo prefix="${vacuum_gripper_prefix}" gripper_link="robot_system_::robot_wrist_3_link">
     <drops_info/>
-  </xacro:vacuum_gripper_gazebo>
+  </xacro:simple_gripper_gazebo>
   <!-- Joints -->
   <joint name="robot_to_carriage" type="fixed">

File: gilbreth_support/urdf/simple_gripper/simple_gripper.gazebo.xacro (robot description, xacro)
@@ -1,5 +1,5 @@
 <?xml version="1.0"?>
 <robot xmlns:xacro="http://www.ros.org/wiki/xacro">
-  <xacro:macro name="vacuum_gripper_gazebo" params="prefix **drops_info gripper_link">
+  <xacro:macro name="simple_gripper_gazebo" params="prefix **drops_info gripper_link">
     <gazebo reference="${prefix}base_link">
       <material>Gazebo/Red</material>

File: gilbreth_support/urdf/simple_gripper/simple_gripper.xacro (robot description, xacro)
@@ -1,10 +1,10 @@
 <?xml version="1.0"?>
 <robot name="vacuum_gripper" xmlns:xacro="http://www.ros.org/wiki/xacro">
-  <arg name="prefix" default="vacuum_gripper_"/>
+  <arg name="prefix" default="simple_gripper_"/>
   <!-- URDF -->
-  <xacro:include filename="$(find gilbreth_support)/urdf/vacuum_gripper/vacuum_gripper.urdf.xacro"/>
+  <xacro:include filename="$(find gilbreth_support)/urdf/simple_gripper/simple_gripper.urdf.xacro"/>
   <xacro:vacuum_gripper_urdf prefix="$(arg prefix)"/>
   <!-- Gazebo -->
-  <xacro:include filename="$(find gilbreth_support)/urdf/vacuum_gripper/vacuum_gripper.gazebo.xacro"/>
+  <xacro:include filename="$(find gilbreth_support)/urdf/simple_gripper/simple_gripper.gazebo.xacro"/>
   <xacro:vacuum_gripper_gazebo prefix="$(arg prefix)" gripper_link="${prefix}::${prefix}tool0">
     <drops_info/>
